File: RF_Transiever/RF_Transiever.kicad_sch (KiCad schematic)
At the start: 48 parts, among them J1 Conn_01x08_Pin, J2 Conn_01x08_Pin, J3 CON-SMA-EDGE-SRP, U1 SX1278, U2 RFSW6024, U3 NC7SZ04M5X

Commit message: v1.0.0
Connections:
- net at C2.1, U1.2 (VR_ANA): no longer C1.1, U1.4 (VR_DIG)
- new net: C1.1, U1.4 (VR_DIG)
Other:
- moved on the sheet: C1, C2
Changed lines of the file:
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@@
 	)
 	(junction
-		(at 201.93 57.15)
-		(diameter 0)
-		(color 0 0 0 0)
-	)
-	(junction
 		(at 189.23 172.72)
 		(diameter 0)
@@
 	)
 	(junction
-		(at 190.5 48.26)
-		(diameter 0)
-		(color 0 0 0 0)
-	)
-	(junction
 		(at 256.54 76.2)
 		(diameter 0)
@@
 	)
 	(junction
-		(at 194.31 48.26)
-		(diameter 0)
-		(color 0 0 0 0)
-	)
-	(junction
 		(at 288.29 76.2)
 		(diameter 0)
@@
 	(wire
 		(pts
-			(xy 194.31 57.15) (xy 201.93 57.15)
+			(xy 340.36 163.83) (xy 347.98 163.83)
 		)
 		(stroke
@@
 	(wire
 		(pts
-			(xy 340.36 163.83) (xy 347.98 163.83)
+			(xy 269.24 76.2) (xy 269.24 77.47)
 		)
 		(stroke
@@
 	(wire
 		(pts
-			(xy 269.24 76.2) (xy 269.24 77.47)
+			(xy 182.88 48.26) (xy 185.42 48.26)
 		)
 		(stroke
@@
 	(wire
 		(pts
-			(xy 182.88 48.26) (xy 185.42 48.26)
+			(xy 316.23 215.9) (xy 316.23 218.44)
 		)
 		(stroke
@@
 	(wire
 		(pts
-			(xy 316.23 215.9) (xy 316.23 218.44)
+			(xy 207.01 45.72) (xy 207.01 48.26)
 		)
 		(stroke
@@
 	(wire
 		(pts
-			(xy 190.5 48.26) (xy 194.31 48.26)
+			(xy 187.96 45.72) (xy 207.01 45.72)
 		)
 		(stroke
@@
 	(wire
 		(pts
+			(xy 194.31 46.99) (xy 194.31 48.26)
+		)
+		(stroke
+			(width 0)
+			(type default)
+		)
+	)
+	(wire
+		(pts
 			(xy 288.29 85.09) (xy 288.29 86.36)
 		)
@@
 	(wire
 		(pts
-			(xy 201.93 57.15) (xy 207.01 57.15)
-		)
-		(stroke
-			(width 0)
-			(type default)
-		)
-	)
-	(wire
-		(pts
 			(xy 270.51 43.18) (xy 275.59 43.18)
 		)
@@
 	(wire
 		(pts
-			(xy 207.01 55.88) (xy 207.01 57.15)
+			(xy 207.01 55.88) (xy 207.01 58.42)
 		)
 		(stroke
@@
 	(wire
 		(pts
-			(xy 194.31 55.88) (xy 194.31 57.15)
-		)
-		(stroke
-			(width 0)
-			(type default)
-		)
-	)
-	(wire
-		(pts
-			(xy 194.31 48.26) (xy 207.01 48.26)
-		)
-		(stroke
-			(width 0)
-			(type default)
-		)
-	)
-	(wire
-		(pts
 			(xy 55.88 93.98) (xy 72.39 93.98)
 		)
@@
 	(wire
 		(pts
-			(xy 190.5 48.26) (xy 190.5 60.96)
-		)
-		(stroke
-			(width 0)
-			(type default)
-		)
-	)
-	(wire
-		(pts
 			(xy 259.08 64.77) (xy 254 64.77)
 		)
@@
 	(wire
 		(pts
-			(xy 187.96 60.96) (xy 187.96 48.26)
+			(xy 187.96 60.96) (xy 187.96 45.72)
 		)
 		(stroke
@@
 	(wire
 		(pts
+			(xy 190.5 60.96) (xy 190.5 46.99)
+		)
+		(stroke
+			(width 0)
+			(type default)
+		)
+	)
+	(wire
+		(pts
 			(xy 55.88 95.25) (xy 55.88 93.98)
 		)
@@
 	(wire
 		(pts
-			(xy 201.93 57.15) (xy 201.93 58.42)
+			(xy 194.31 55.88) (xy 194.31 58.42)
 		)
 		(stroke
@@
 	(wire
 		(pts
-			(xy 165.1 83.82) (xy 170.18 83.82)
+			(xy 190.5 46.99) (xy 194.31 46.99)
 		)
 		(stroke
@@
 	(wire
 		(pts
-			(xy 360.68 158.75) (xy 360.68 161.29)
+			(xy 165.1 83.82) (xy 170.18 83.82)
 		)
 		(stroke
@@
 	(wire
 		(pts
-			(xy 52.07 200.66) (xy 64.77 200.66)
+			(xy 360.68 158.75) (xy 360.68 161.29)
 		)
 		(stroke
@@
 	(wire
 		(pts
-			(xy 151.13 57.15) (xy 157.48 57.15)
+			(xy 52.07 200.66) (xy 64.77 200.66)
 		)
 		(stroke
@@
 	(wire
 		(pts
-			(xy 144.78 55.88) (xy 144.78 57.15)
+			(xy 151.13 57.15) (xy 157.48 57.15)
 		)
 		(stroke
@@
 	(wire
 		(pts
-			(xy 283.21 43.18) (xy 287.02 43.18)
+			(xy 144.78 55.88) (xy 144.78 57.15)
 		)
 		(stroke
@@
 	(wire
 		(pts
-			(xy 187.96 48.26) (xy 190.5 48.26)
+			(xy 283.21 43.18) (xy 287.02 43.18)
 		)
 		(stroke
@@
 	)
 	(symbol
+		(lib_id "power:GND")
+		(at 207.01 58.42 0)
+		(unit 1)
+		(exclude_from_sim no)
+		(in_bom yes)
+		(on_board yes)
+		(dnp no)
+		(property "Reference" "#PWR023"
+			(at 207.01 64.77 0)
+			(effects
+				(font
+					(size 1.27 1.27)
+				)
+				(hide yes)
+			)
+		)
+		(property "Value" "GND"
+			(at 207.01 62.23 0)
+			(effects
+				(font
+					(size 1.27 1.27)
+				)
+			)
+		)
+		(property "Footprint" ""
+			(at 207.01 58.42 0)
+			(effects
+				(font
+					(size 1.27 1.27)
+				)
+				(hide yes)
+			)
+		)
+		(property "Datasheet" ""
+			(at 207.01 58.42 0)
+			(effects
+				(font
+					(size 1.27 1.27)
+				)
+				(hide yes)
+			)
+		)
+		(property "Description" "Power symbol creates a global label with name \"GND\" , ground"
+			(at 207.01 58.42 0)
+			(effects
+				(font
+					(size 1.27 1.27)
+				)
+				(hide yes)
+			)
+		)
+		(pin "1"
+		)
+		(instances
+			(project "RF_Transiever"
+				(path "/dd17954e-3bc3-49ba-a493-70ae577e40b8"
+					(reference "#PWR023")
+					(unit 1)
+				)
+			)
+		)
+	)
+	(symbol
 		(lib_id "Device:C")
 		(at 132.08 52.07 0)
@@
 	(symbol
 		(lib_id "power:GND")
-		(at 201.93 58.42 0)
+		(at 194.31 58.42 0)
 		(unit 1)
 		(exclude_from_sim no)
@@
 		(dnp no)
 		(property "Reference" "#PWR07"
-			(at 201.93 64.77 0)
+			(at 194.31 64.77 0)
 			(effects
 				(font
@@
 		)
 		(property "Value" "GND"
-			(at 201.93 62.23 0)
+			(at 194.31 62.23 0)
 			(effects
 				(font
@@
 		)
 		(property "Footprint" ""
-			(at 201.93 58.42 0)
+			(at 194.31 58.42 0)
 			(effects
 				(font
@@
 		)
 		(property "Datasheet" ""
-			(at 201.93 58.42 0)
+			(at 194.31 58.42 0)
 			(effects
 				(font
@@
 		)
 		(property "Description" "Power symbol creates a global label with name \"GND\" , ground"
-			(at 201.93 58.42 0)
+			(at 194.31 58.42 0)
 			(effects
 				(font
@@
 		)
 		(instances
-			(project ""
+			(project "RF_Transiever"
 				(path "/dd17954e-3bc3-49ba-a493-70ae577e40b8"
 					(reference "#PWR07")
@@
 	(symbol
 		(lib_id "Device:C")
-		(at 207.01 52.07 0)
+		(at 194.31 52.07 0)
 		(unit 1)
 		(exclude_from_sim no)
@@
 		(fields_autoplaced yes)
 		(property "Reference" "C1"
-			(at 210.82 50.7999 0)
+			(at 198.12 50.7999 0)
 			(effects
 				(font
@@
 		)
 		(property "Value" "100nF"
-			(at 210.82 53.3399 0)
+			(at 198.12 53.3399 0)
 			(effects
 				(font
@@
 		)
 		(property "Footprint" "Capacitor_SMD:C_0402_1005Metric"
-			(at 207.9752 55.88 0)
+			(at 195.2752 55.88 0)
 			(effects
 				(font
@@
 		)
 		(property "Datasheet" "~"
-			(at 207.01 52.07 0)
+			(at 194.31 52.07 0)
 			(effects
 				(font
@@
 		)
 		(property "Description" "Unpolarized capacitor"
-			(at 207.01 52.07 0)
+			(at 194.31 52.07 0)
 			(effects
 				(font
@@
 		)
 		(instances
-			(project ""
+			(project "RF_Transiever"
 				(path "/dd17954e-3bc3-49ba-a493-70ae577e40b8"
 					(reference "C1")
@@
 	(symbol
 		(lib_id "Device:C")
-		(at 194.31 52.07 0)
+		(at 207.01 52.07 0)
 		(unit 1)
 		(exclude_from_sim no)
@@
 		(fields_autoplaced yes)
 		(property "Reference" "C2"
-			(at 198.12 50.7999 0)
+			(at 210.82 50.7999 0)
 			(effects
 				(font
@@
 		)
 		(property "Value" "100nF"
-			(at 198.12 53.3399 0)
+			(at 210.82 53.3399 0)
 			(effects
 				(font
@@
 		)
 		(property "Footprint" "Capacitor_SMD:C_0402_1005Metric"
-			(at 195.2752 55.88 0)
+			(at 207.9752 55.88 0)
 			(effects
 				(font
@@
 		)
 		(property "Datasheet" "~"
-			(at 194.31 52.07 0)
+			(at 207.01 52.07 0)
 			(effects
 				(font
@@
 		)
 		(property "Description" "Unpolarized capacitor"
-			(at 194.31 52.07 0)
+			(at 207.01 52.07 0)
 			(effects
 				(font
